File: elderstep.brd (EAGLE design)
At the start: 46.7 x 33 mm, 27 parts, among them CN2 JSTPH, U1 MCP73831T-2ACI/OT

Commit message: revA
Parts:
- moved CN2 0.76 mm to (95.8, 5.08)
Routing:
- net GND: track 227.3 -> 211.7 mm
- net VCC: track 77.2 -> 72.5 mm
- net VBAT: track 53.2 -> 50.6 mm
- added copper zone on layer 1, net GND
Other:
- board size 46.7 x 33 mm -> 41.7 x 32 mm
- board text added: "10/04/17"
- board text added: "ElderStep"
- board text added: "revA"
